Commit message: Implemented Lidar VLP-16 as seen in abb-crafter project. Understanding ist tbd

File: src/localisation_gazebo/robot/lidar.xacro (robot description, xacro)
@@ -14,5 +14,5 @@
    <parent link="base_footprint" />
     <child link="base_link" />
-    <origin xyz="0 0 0.67" rpy="0 0 0" />
+    <origin xyz="10 10 0.67" rpy="0 0 0" />
   </joint>
   <link name="base_link" >
@@ -36,5 +36,6 @@
   </link>
   <xacro:include filename="$(find velodyne_description)/urdf/VLP-16.urdf.xacro"/>
-  <xacro:VLP-16 parent="base_link" name="velodyne" topic="/velodyne_points" organize_cloud="${organize_cloud}" hz="10" samples="440" gpu="${gpu}">
+  <xacro:VLP-16 parent="base_link" name="velodyne" topic="/velodyne_points" organize_cloud="${organize_cloud}" hz="10" samples="440" gpu="${gpu}" max_range="100" min_angle="-${1.5708}" max_angle="${1.5708}">
     <origin xyz="0 0 0.4" rpy="0 0 0" />
   </xacro:VLP-16>
+</robot>

Commit message: move_sim angepasst, localisation header und file hinzugefügt, CMakeLists entsprechend angepasst, lidar verändert so dass 360Grad abtastung, rviz file geändert um nur einen LIDAR Sensor anzuzeigen (Überbleibsel altes Projekt)

File: src/localisation_gazebo/robot/lidar.xacro (robot description, xacro)
@@ -14,5 +14,5 @@
    <parent link="base_footprint" />
     <child link="base_link" />
-    <origin xyz="10 10 0.67" rpy="0 0 0" />
+    <origin xyz="0 10 0.67" rpy="0 0 0" />
   </joint>
   <link name="base_link" >
@@ -36,5 +36,5 @@
   </link>
   <xacro:include filename="$(find velodyne_description)/urdf/VLP-16.urdf.xacro"/>
-  <xacro:VLP-16 parent="base_link" name="velodyne" topic="/velodyne_points" organize_cloud="${organize_cloud}" hz="10" samples="440" gpu="${gpu}" max_range="100" min_angle="-${1.5708}" max_angle="${1.5708}">
+  <xacro:VLP-16 parent="base_link" name="velodyne" topic="/velodyne_points" organize_cloud="${organize_cloud}" hz="10" samples="440" gpu="${gpu}" max_range="100" min_angle="-${M_PI}" max_angle="${M_PI}">
     <origin xyz="0 0 0.4" rpy="0 0 0" />
   </xacro:VLP-16>

Commit message: Slight changes. More for getting understanding of abb ROS Nodes.

File: src/localisation_gazebo/robot/lidar.xacro (robot description, xacro)
@@ -14,19 +14,19 @@
    <parent link="base_footprint" />
     <child link="base_link" />
-    <origin xyz="0 10 0.67" rpy="0 0 0" />
+    <origin xyz="0 10 1.25" rpy="0 0 0" />
   </joint>
   <link name="base_link" >
     <visual>
       <geometry>
-        <box size="0.5 0.5 0.1" />
+        <box size="0.1 0.1 2.5" />
       </geometry>
     </visual>
     <collision>
       <geometry>
-        <box size="0.5 0.5 0.1" />
+        <box size="0.1 0.1 2.5" />
       </geometry>
     </collision>
     <inertial>
-      <origin xyz="0 0 0"/>
+      <origin xyz="0 0 1.25"/>
       <mass value="10"/>
       <inertia ixx="3.0" ixy="0.0" ixz="0.0"
@@ -37,5 +37,5 @@
   <xacro:include filename="$(find velodyne_description)/urdf/VLP-16.urdf.xacro"/>
   <xacro:VLP-16 parent="base_link" name="velodyne" topic="/velodyne_points" organize_cloud="${organize_cloud}" hz="10" samples="440" gpu="${gpu}" max_range="100" min_angle="-${M_PI}" max_angle="${M_PI}">
-    <origin xyz="0 0 0.4" rpy="0 0 0" />
+    <origin xyz="0 0 1.25" rpy="0 0 0" />
   </xacro:VLP-16>
 </robot>

Commit message: Erste Tests für Filterung. Ergebnisse auskommentiert

File: src/localisation_gazebo/robot/lidar.xacro (robot description, xacro)
@@ -14,5 +14,5 @@
    <parent link="base_footprint" />
     <child link="base_link" />
-    <origin xyz="0 10 1.25" rpy="0 0 0" />
+    <origin xyz="5 10 1.25" rpy="0 0 0" />
   </joint>
   <link name="base_link" >
@@ -36,5 +36,5 @@
   </link>
   <xacro:include filename="$(find velodyne_description)/urdf/VLP-16.urdf.xacro"/>
-  <xacro:VLP-16 parent="base_link" name="velodyne" topic="/velodyne_points" organize_cloud="${organize_cloud}" hz="10" samples="440" gpu="${gpu}" max_range="100" min_angle="-${M_PI}" max_angle="${M_PI}">
+  <xacro:VLP-16 parent="base_link" name="velodyne" topic="/velodyne_points" organize_cloud="${organize_cloud}" hz="10" samples="500" gpu="${gpu}" max_range="100" min_angle="-${M_PI}" max_angle="${M_PI}">
     <origin xyz="0 0 1.25" rpy="0 0 0" />
   </xacro:VLP-16>

Commit message: Struktur verändert: Header Orientierte Programmierung. Clustering-Algorithmus eingefügt, kann über message ausglesen werden. Test-Files aus Projektstruktur entfernt.

File: src/localisation_gazebo/robot/lidar.xacro (robot description, xacro)
@@ -14,5 +14,5 @@
    <parent link="base_footprint" />
     <child link="base_link" />
-    <origin xyz="5 10 1.25" rpy="0 0 0" />
+    <origin xyz="20 10 1.25" rpy="0 0 0" />
   </joint>
   <link name="base_link" >

Commit message: diverse messages ergänzt und code aufgeräumt. Funktionen hinzugefügt (vergleichen Dreiecke, prüfen ob Punkt in Dreieck liegt). Move Sim kann jetzt mit Parameteren für x und y position gefüttert werden

File: src/localisation_gazebo/robot/lidar.xacro (robot description, xacro)
@@ -14,5 +14,5 @@
    <parent link="base_footprint" />
     <child link="base_link" />
-    <origin xyz="20 10 1.25" rpy="0 0 0" />
+    <origin xyz="0 0 1.25" rpy="0 0 0" />
   </joint>
   <link name="base_link" >
